File: DJI_to_xt30.kicad_pcb (KiCad board)
At the start: 2 copper layers, 52.8 x 18.6 mm, 6 parts, among them J1 Conn_01x10_Male, J2 Conn_01x02_Female

Commit message: Updated to kicad 7, Added image.
Other:
- net class Default removed
